File: Mobile_Camera.kicad_sch (KiCad schematic)
At the start: 22 parts, among them J1 SWD_header, J2 DVP_24_pin, J3 Micro_SD_card, SW1 Switch_reset, SW2 Switch_power_on, U1 STM32H753VIT6, Y1 Crystal

Commit message: Assign antenna, camera and crystal footprint
Parts:
- J2: footprint (none) -> Connector_FFC-FPC:TE_2-1734839-4_1x24-1MP_P0.5mm_Horizontal
- Y1: footprint (none) -> Crystal:Crystal_SMD_SeikoEpson_TSX3225-4Pin_3.2x2.5mm_HandSoldering
Changed lines of the file:
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@@
       (effects (font (size 1.27 1.27)) (justify left))
     )
-    (property "Footprint" "" (at 140.97 101.6 0)
+    (property "Footprint" "Crystal:Crystal_SMD_SeikoEpson_TSX3225-4Pin_3.2x2.5mm_HandSoldering" (at 140.97 101.6 0)
       (effects (font (size 1.27 1.27)) hide)
     )
@@
       (effects (font (size 1.27 1.27)) (justify left))
     )
-    (property "Footprint" "" (at 184.15 58.42 0)
-      (effects (font (size 1.27 1.27)) hide)
-    )
+    (property "Footprint" "Connector_FFC-FPC:TE_2-1734839-4_1x24-1MP_P0.5mm_Horizontal" (at 184.15 58.42 0)
+      (effects (font (size 1.27 1.27)) hide)
+    )
