File: Mobile_Camera.kicad_pcb (KiCad board)
At the start: 2 copper layers, 62 x 87 mm, 85 parts, among them J1 SWD_header, J2 DVP_24_pin, J3 Micro_SD_card, J4 Antenna_connector, J5 Micro_SIM_card, J6 USB_C_receptacle, Q1 Q_NPN, SW1 SW_Power_On, SW2 SW_Reset, U1 STM32H753VIT6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

Commit message: Complete the PCB design
Parts:
- J4: footprint Connector_Coaxial:U.FL_Molex_MCRF_73412-0110_Vertical -> Connector_Coaxial:U.FL_Hirose_U.FL-R-SMT-1_Vertical
- moved J4 0.48 mm to (107.0, 47.5), turned to -90 degrees
Changed lines of the file:
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@@
       (outputformat 1)
       (mirror false)
-      (drillshape 1)
+      (drillshape 0)
       (scaleselection 1)
-      (outputdirectory "")
+      (outputdirectory "../Pliki_CAM/")
     )
   )
@@
     (fp_line (start 2.25 1.6) (end -2.25 1.6)
       (stroke (width 0.1) (type solid)) (layer "F.Fab"))
-    (pad "1" smd roundrect (at -2.225 0 270) (size 1.3 3.4) (layers "F.Cu" "F.Paste" "F.Mask") (roundrect_rratio 0.192308)
+    (pad "1" smd roundrect (at -2.225 0 270) (size 1.3 3.4) (layers "F.Cu" "F.Paste" "F.Mask") (roundrect_rratio 0.1923076923)
       (net 28 "Net-(F1-Pad1)") (pintype "passive"))
-    (pad "2" smd roundrect (at 2.225 0 270) (size 1.3 3.4) (layers "F.Cu" "F.Paste" "F.Mask") (roundrect_rratio 0.192308)
+    (pad "2" smd roundrect (at 2.225 0 270) (size 1.3 3.4) (layers "F.Cu" "F.Paste" "F.Mask") (roundrect_rratio 0.1923076923)
       (net 13 "+5V") (pintype "passive"))
     (model "${KICAD6_3DMODEL_DIR}/Fuse.3dshapes/Fuse_1812_4532Metric.wrl"
@@
     )
   )
-  (footprint "Connector_Coaxial:U.FL_Molex_MCRF_73412-0110_Vertical" (layer "F.Cu")
-    (at 107 48 180)
-    (descr "Molex Microcoaxial RF Connectors (MCRF), mates Hirose U.FL, (http://www.molex.com/pdm_docs/sd/734120110_sd.pdf)")
-    (tags "mcrf hirose ufl u.fl microcoaxial")
+  (footprint "Connector_Coaxial:U.FL_Hirose_U.FL-R-SMT-1_Vertical" (layer "F.Cu")
+    (at 107 47.525 -90)
+    (descr "Hirose U.FL Coaxial https://www.hirose.com/product/en/products/U.FL/U.FL-R-SMT-1%2810%29/")
+    (tags "Hirose U.FL Coaxial")
     (property "Sheetfile" "sim.kicad_sch")
     (property "Sheetname" "SIM")
@@
     (property "ki_keywords" "BNC SMA SMB SMC LEMO coaxial connector CINCH RCA")
     (attr smd)
-    (fp_text reference "J4" (at 0 3.5) (layer "F.SilkS")
+    (fp_text reference "J4" (at 0.475 -3.2 90) (layer "F.SilkS")
         (effects (font (size 1 1) (thickness 0.15)))
     )
-    (fp_text value "Antenna_connector" (at 0 -3.302) (layer "F.Fab")
+    (fp_text value "Antenna_connector" (at 0.475 3.2 90) (layer "F.Fab")
         (effects (font (size 1 1) (thickness 0.15)))
     )
-    (fp_text user "${REFERENCE}" (at 0 3.5) (layer "F.Fab")
-        (effects (font (size 1 1) (thickness 0.15)))
+    (fp_text user "${REFERENCE}" (at 0.475 0) (layer "F.Fab")
+        (effects (font (size 0.6 0.6) (thickness 0.09)))
     )
-    (fp_line (start -1.5 -1.5) (end -0.7 -1.5)
-      (stroke (width 0.12) (type solid)) (layer "F.SilkS"))
-    (fp_line (start -1.5 -1.3) (end -1.5 -1.5)
-      (stroke (width 0.12) (type solid)) (layer "F.SilkS"))
-    (fp_line (start -1.3 1.5) (end -1.5 1.3)
-      (stroke (width 0.12) (type solid)) (layer "F.SilkS"))
-    (fp_line (start -0.7 1.5) (end -1.3 1.5)
-      (stroke (width 0.12) (type solid)) (layer "F.SilkS"))
-    (fp_line (start -0.7 1.5) (end -0.7 2)
+    (fp_line (start -0.885 -1.4) (end -0.885 -0.76)
       (stroke (width 0.12) (type solid)) (layer "F.SilkS"))
-    (fp_line (start 0.7 -1.5) (end 1.5 -1.5)
+    (fp_line (start -0.885 -0.76) (end -1.515 -0.76)
       (stroke (width 0.12) (type solid)) (layer "F.SilkS"))
-    (fp_line (start 0.7 1.5) (end 0.7 2)
+    (fp_line (start -0.885 1.4) (end -0.885 0.76)
       (stroke (width 0.12) (type solid)) (layer "F.SilkS"))
-    (fp_line (start 1.5 -1.5) (end 1.5 -1.3)
+    (fp_line (start 1.835 -1.35) (end 1.835 1.35)
       (stroke (width 0.12) (type solid)) (layer "F.SilkS"))
-    (fp_line (start 1.5 1.3) (end 1.5 1.5)
-      (stroke (width 0.12) (type solid)) (layer "F.SilkS"))
-    (fp_line (start 1.5 1.5) (end 0.7 1.5)
-      (stroke (width 0.12) (type solid)) (layer "F.SilkS"))
-    (fp_line (start -2.5 -2.5) (end -2.5 2.5)
+    (fp_line (start -2.02 1) (end -2.02 -1)
+      (stroke (width 0.05) (type solid)) (layer "F.CrtYd"))
+    (fp_line (start -1.32 -1.8) (end -1.12 -1.8)
+      (stroke (width 0.05) (type solid)) (layer "F.CrtYd"))
+    (fp_line (start -1.32 -1) (end -2.02 -1)
+      (stroke (width 0.05) (type solid)) (layer "F.CrtYd"))
+    (fp_line (start -1.32 -1) (end -1.32 -1.8)
+      (stroke (width 0.05) (type solid)) (layer "F.CrtYd"))
+    (fp_line (start -1.32 1) (end -2.02 1)
+      (stroke (width 0.05) (type solid)) (layer "F.CrtYd"))
+    (fp_line (start -1.32 1.8) (end -1.32 1)
+      (stroke (width 0.05) (type solid)) (layer "F.CrtYd"))
+    (fp_line (start -1.32 1.8) (end -1.12 1.8)
+      (stroke (width 0.05) (type solid)) (layer "F.CrtYd"))
+    (fp_line (start -1.12 -1.8) (end -1.12 -2.5)
+      (stroke (width 0.05) (type solid)) (layer "F.CrtYd"))
+    (fp_line (start -1.12 2.5) (end -1.12 1.8)
+      (stroke (width 0.05) (type solid)) (layer "F.CrtYd"))
+    (fp_line (start 2.08 -2.5) (end -1.12 -2.5)
+      (stroke (width 0.05) (type solid)) (layer "F.CrtYd"))
+    (fp_line (start 2.08 -1.8) (end 2.08 -2.5)
+      (stroke (width 0.05) (type solid)) (layer "F.CrtYd"))
+    (fp_line (start 2.08 -1.8) (end 2.28 -1.8)
       (stroke (width 0.05) (type solid)) (layer "F.CrtYd"))
-    (fp_line (start -2.5 2.5) (end 2.5 2.5)
+    (fp_line (start 2.08 1.8) (end 2.28 1.8)
       (stroke (width 0.05) (type solid)) (layer "F.CrtYd"))
-    (fp_line (start 2.5 -2.5) (end -2.5 -2.5)
+    (fp_line (start 2.08 2.5) (end -1.12 2.5)
       (stroke (width 0.05) (type solid)) (layer "F.CrtYd"))
-    (fp_line (start 2.5 2.5) (end 2.5 -2.5)
+    (fp_line (start 2.08 2.5) (end 2.08 1.8)
       (stroke (width 0.05) (type solid)) (layer "F.CrtYd"))
-    (fp_line (start -1.3 -1.3) (end -1.3 1)
+    (fp_line (start 2.28 1.8) (end 2.28 -1.8)
+      (stroke (width 0.05) (type solid)) (layer "F.CrtYd"))
+    (fp_line (start -1.075 0.3) (end -1.075 -0.15)
       (stroke (width 0.1) (type solid)) (layer "F.Fab"))
-    (fp_line (start -1.3 -1.3) (end 1.3 -1.3)
+    (fp_line (start -1.075 0.3) (end -0.825 0.3)
       (stroke (width 0.1) (type solid)) (layer "F.Fab"))
-    (fp_line (start -1.3 1) (end -1 1.3)
+    (fp_line (start -0.925 -0.3) (end -1.075 -0.15)
       (stroke (width 0.1) (type solid)) (layer "F.Fab"))
-    (fp_line (start -1 1.3) (end 1.3 1.3)
+    (fp_line (start -0.925 -0.3) (end -0.825 -0.3)
       (stroke (width 0.1) (type solid)) (layer "F.Fab"))
-    (fp_line (start -0.3 1.3) (end 0 1)
+    (fp_line (start -0.825 -0.3) (end -0.825 -1.3)
       (stroke (width 0.1) (type solid)) (layer "F.Fab"))
-    (fp_line (start 0 1) (end 0.3 1.3)
+    (fp_line (start -0.825 0.3) (end -0.825 1.3)
       (stroke (width 0.1) (type solid)) (layer "F.Fab"))
-    (fp_line (start 1.3 -1.3) (end 1.3 1.3)
+    (fp_line (start -0.425 -1.5) (end -0.425 -1.3)
       (stroke (width 0.1) (type solid)) (layer "F.Fab"))
-    (fp_circle (center 0 0) (end 0 0.05)
-      (stroke (width 0.1) (type solid)) (fill none) (layer "F.Fab"))
-    (fp_circle (center 0 0) (end 0 0.125)
-      (stroke (width 0.1) (type solid)) (fill none) (layer "F.Fab"))
-    (fp_circle (center 0 0) (end 0 0.2)
-      (stroke (width 0.1) (type solid)) (fill none) (layer "F.Fab"))
-    (fp_circle (center 0 0) (end 0.9 0)
-      (stroke (width 0.1) (type solid)) (fill none) (layer "F.Fab"))
-    (pad "1" smd rect (at 0 1.5 180) (size 1 1) (layers "F.Cu" "F.Paste" "F.Mask")
+    (fp_line (start -0.425 -1.5) (end 1.375 -1.5)
+      (stroke (width 0.1) (type solid)) (layer "F.Fab"))
+    (fp_line (start -0.425 -1.3) (end -0.825 -1.3)
+      (stroke (width 0.1) (type solid)) (layer "F.Fab"))
+    (fp_line (start -0.425 1.3) (end -0.825 1.3)
+      (stroke (width 0.1) (type solid)) (layer "F.Fab"))
+    (fp_line (start -0.425 1.5) (end -0.425 1.3)
+      (stroke (width 0.1) (type solid)) (layer "F.Fab"))
+    (fp_line (start -0.425 1.5) (end 1.375 1.5)
+      (stroke (width 0.1) (type solid)) (layer "F.Fab"))
+    (fp_line (start 1.375 -1.5) (end 1.375 -1.3)
+      (stroke (width 0.1) (type solid)) (layer "F.Fab"))
+    (fp_line (start 1.375 1.5) (end 1.375 1.3)
+      (stroke (width 0.1) (type solid)) (layer "F.Fab"))
+    (fp_line (start 1.775 -1.3) (end 1.375 -1.3)
+      (stroke (width 0.1) (type solid)) (layer "F.Fab"))
+    (fp_line (start 1.775 -1.3) (end 1.775 1.3)
+      (stroke (width 0.1) (type solid)) (layer "F.Fab"))
+    (fp_line (start 1.775 1.3) (end 1.375 1.3)
+      (stroke (width 0.1) (type solid)) (layer "F.Fab"))
+    (pad "1" smd rect (at -1.05 0 270) (size 1.05 1) (layers "F.Cu" "F.Paste" "F.Mask")
       (net 2 "GND") (pinfunction "In") (pintype "passive"))
-    (pad "2" smd rect (at -1.475 0 180) (size 1.05 2.2) (layers "F.Cu" "F.Paste" "F.Mask")
+    (pad "2" smd rect (at 0.475 -1.475 270) (size 2.2 1.05) (layers "F.Cu" "F.Paste" "F.Mask")
       (net 57 "/SIM/GSM_ANT") (pinfunction "Ext") (pintype "passive"))
-    (pad "2" smd rect (at 0 -1.5 180) (size 1 1) (layers "F.Cu" "F.Paste" "F.Mask")
+    (pad "2" smd rect (at 0.475 1.475 270) (size 2.2 1.05) (layers "F.Cu" "F.Paste" "F.Mask")
       (net 57 "/SIM/GSM_ANT") (pinfunction "Ext") (pintype "passive"))
-    (pad "2" smd rect (at 1.475 0 180) (size 1.05 2.2) (layers "F.Cu" "F.Paste" "F.Mask")
-      (net 57 "/SIM/GSM_ANT") (pinfunction "Ext") (pintype "passive"))
-    (model "${KICAD6_3DMODEL_DIR}/Connector_Coaxial.3dshapes/U.FL_Molex_MCRF_73412-0110_Vertical.wrl"
-      (offset (xyz 0 0 0))
+    (model "${KICAD6_3DMODEL_DIR}/Connector_Coaxial.3dshapes/U.FL_Hirose_U.FL-R-SMT-1_Vertical.wrl"
+      (offset (xyz 0.4749999928 0 0))
       (scale (xyz 1 1 1))
       (rotate (xyz 0 0 0))
